Commit message: Add launch & gazebo param for go2
Signed-off-by: C88-YQ <1409947012@qq.com>

File: b2w_sim/go2_description/urdf/go2_description.urdf (robot description, URDF)
Before this commit: robot go2_description, 42 links, 41 joints
Links:
- added link collision_plate, mass 0.05; collision box size=0.47 0.20 0.02; visual box size=0.45 0.18 0.02
- added link realsense_camera, mass 0.08; collision box size=0.09 0.025 0.025
Joints:
- added joint base_to_collision_plate: type fixed, parent base, child collision_plate, origin xyz=0.02 0 0.06 rpy=0 0 0, axis 0 0 0
- added joint base_to_realsense_camera: type fixed, parent base, child realsense_camera, origin xyz=0.32715 0 0.10 rpy=0 0 0, axis 0 0 0
